Commit message: RPLidar added to package

File: model_lidar/description/model.urdf.xacro (robot description, xacro)
@@ -2,3 +2,4 @@
 <robot xmlns:xacro="http://www.ros.org/wiki/xacro"  name="robot_slam">
     <xacro:include filename="model_main.xacro" />
+    <xacro:include filename="lidar.xacro" />
 </robot>

File: model_lidar/description/model_main.xacro (robot description, xacro)
@@ -38,30 +38,4 @@
             <origin xyz="0.15 0 0.075" rpy="0 0 0"/>
         </xacro:inertial_box>
-    </link>
-    <!--lidar-->
-    <joint name="lidarr_joint" type="fixed">
-        <parent link="base_link"/>
-        <child link="lidarr"/>
-        <origin xyz="0 0 0.225" rpy="0 0 0"/>
-    </joint>
-        <link name="lidarr">
-        <visual>
-            <geometry>
-                <cylinder radius="0.025" length="0.07"/>
-            </geometry>
-            <material name="blue">
-                <color rgba="0.0 0.0 1.0 1.0"/>
-            </material>
-        </visual>
-        <collision>
-            <geometry>
-                <cylinder radius="0.025" length="0.07"/>
-            </geometry>
-        </collision>
-        <inertial>
-            <mass value="0.2"/>
-            <origin xyz="0 0 0.225" />
-            <inertia ixx="0.01" ixy="0.0" ixz="0.0" iyy="0.01" iyz="0.0" izz="0.01"/>
-        </inertial>
     </link>
     <!-- LEFT WHEEL LINK -->
