Commit message: fixed slam_toolbox and driving

File: robot_slam/description/lidar.xacro (robot description, xacro)
@@ -6,5 +6,5 @@
         <origin xyz="0 0 0.25" rpy="0 0 0"/>
     </joint>
-        <link name="lidar">
+    <link name="lidar">
         <visual>
             <geometry>
@@ -26,3 +26,3 @@
         </inertial>
     </link>
-    </robot>
+</robot>

File: robot_slam/description/model.urdf.xacro (robot description, xacro)
@@ -4,3 +4,17 @@
     <xacro:include filename="lidar.xacro" />
     <xacro:include filename="ros2_control.xacro" />
+    <link name="odom"/>
+    <joint name="odom_to_base_link" type="fixed">
+        <parent link="odom"/>
+        <child link="base_link"/>
+        <origin xyz="0 0 0" rpy="0 0 0"/>
+    </joint>
+    <link name="laser">
+      <!-- Laser sensor properties -->
+    </link>
+    <joint name="laser_joint" type="fixed">
+      <parent link="base_link"/>
+      <child link="laser"/>
+      <origin xyz="0 0 0.1" rpy="0 0 0"/>
+    </joint>
 </robot>

File: robot_slam/description/model_main.xacro (robot description, xacro)
@@ -1,5 +1,7 @@
 <?xml version="1.0"?>
-<robot xmlns:xacro="http://www.ros.org/wiki/xacro" >
+<robot name="RealRobot" xmlns:xacro="http://www.ros.org/wiki/xacro" >
     <xacro:include filename="inertial_macros.xacro"/>
+    <xacro:include filename="$(find robot_slam)/description/lidar.xacro"/>
+    <xacro:include filename="$(find robot_slam)/description/ros2_control.xacro"/>
     <material name="white">
         <color rgba="1 1 1 1" />
@@ -16,4 +18,17 @@
     <link name="base_link">
     </link>
+    <joint name="base_footprint_joint" type="fixed">
+        <parent link="base_link"/>
+        <child link="base_footprint"/>
+        <origin xyz="0 0 0" rpy="0 0 0"/>
+    </joint>
+    <link name="base_footprint">
+    </link>
+    <link name="odom"/>
+    <joint name="odom_to_base_link" type="fixed">
+        <parent link="odom"/>
+        <child link="base_link"/>
+        <origin xyz="0 0 0" rpy="0 0 0"/>
+    </joint>
     <joint name="container_joint" type="fixed">
         <parent link="base_link"/>
@@ -39,4 +54,19 @@
         </xacro:inertial_box>
     </link>
+    <!-- Laser Link -->
+    <link name="laser">
+        <visual>
+            <geometry>
+                <cylinder radius="0.02" length="0.01"/>
+            </geometry>
+            <material name="black"/>
+        </visual>
+    </link>
+    <!-- Laser Joint -->
+    <joint name="laser_joint" type="fixed">
+        <parent link="base_link"/>
+        <child link="laser"/>
+        <origin xyz="0 0 0.1" rpy="0 0 0"/>
+    </joint>
     <!-- LEFT WHEEL LINK -->
     <joint name="left_wheel_joint" type="continuous">
@@ -128,3 +158,32 @@
         </xacro:inertial_sphere>
     </link>
+    <!-- ros2_control configuration -->
+    <ros2_control name="RealRobot" type="system">
+        <hardware>
+            <plugin>diffdrive_arduino/DiffDriveArduinoHardware</plugin>
+            <param name="left_wheel_name">left_wheel_joint</param>
+            <param name="right_wheel_name">right_wheel_joint</param>
+            <param name="loop_rate">30</param>
+            <param name="device">/dev/serial/by-path/platform-fd500000.pcie-pci-0000:01:00.0-usb-0:1.3:1.0-port0</param>
+            <param name="baud_rate">57600</param>
+            <param name="timeout_ms">1000</param>
+            <param name="enc_counts_per_rev">242</param>
+        </hardware>
+        <joint name="left_wheel_joint">
+            <command_interface name="velocity">
+                <param name="min">-50</param>
+                <param name="max">50</param>
+            </command_interface>
+            <state_interface name="position"/>
+            <state_interface name="velocity"/>
+        </joint>
+        <joint name="right_wheel_joint">
+            <command_interface name="velocity">
+                <param name="min">-50</param>
+                <param name="max">50</param>
+            </command_interface>
+            <state_interface name="position"/>
+            <state_interface name="velocity"/>
+        </joint>
+    </ros2_control>
 </robot>

File: robot_slam/description/ros2_control.xacro (robot description, xacro)
@@ -4,9 +4,9 @@
         <ros2_control name="RealRobot" type="system">
             <hardware>
-                <plugin>motor_controll/DiffDriveArduinoHardware</plugin>
+                <plugin>diffdrive_arduino/DiffDriveArduinoHardware</plugin>
                 <param name="left_wheel_name">left_wheel_joint</param>
                 <param name="right_wheel_name">right_wheel_joint</param>
                 <param name="loop_rate">30</param>
-                <param name="device">/dev/serial/by-path/platform-fd500000.pcie-pci-0000:01:00.0-usb-0:1.3:1.0-port0 </param>
+                <param name="device">/dev/serial/by-path/platform-fd500000.pcie-pci-0000:01:00.0-usb-0:1.3:1.0-port0</param>
                 <param name="baud_rate">57600</param>
                 <param name="timeout_ms">1000</param>
