Commit message: nav+map

File: robot_slam/description/model.urdf.xacro (robot description, xacro)
@@ -1,20 +1,9 @@
 <?xml version="1.0"?>
-<robot xmlns:xacro="http://www.ros.org/wiki/xacro"  name="robot_slam">
-    <xacro:include filename="model_main.xacro" />
-    <xacro:include filename="lidar.xacro" />
-    <xacro:include filename="ros2_control.xacro" />
-    <link name="odom"/>
-    <joint name="odom_to_base_link" type="fixed">
-        <parent link="odom"/>
-        <child link="base_link"/>
-        <origin xyz="0 0 0" rpy="0 0 0"/>
-    </joint>
-    <link name="laser">
-      <!-- Laser sensor properties -->
-    </link>
-    <joint name="laser_joint" type="fixed">
-      <parent link="base_link"/>
-      <child link="laser"/>
-      <origin xyz="0 0 0.1" rpy="0 0 0"/>
-    </joint>
+<robot xmlns:xacro="http://www.ros.org/wiki/xacro" name="robot_slam">
+    <xacro:arg name="use_ros2_control" default="true"/>
+    <xacro:arg name="sim_mode" default="false"/>
+    <xacro:include filename="model_main.xacro"/>
+    <!-- Include ros2_control configuration -->
+    <xacro:include filename="ros2_control.xacro"/>
+    <xacro:ros2_control_robot use_ros2_control="$(arg use_ros2_control)" sim_mode="$(arg sim_mode)"/>
 </robot>

File: robot_slam/description/model_main.xacro (robot description, xacro)
@@ -2,6 +2,4 @@
 <robot name="RealRobot" xmlns:xacro="http://www.ros.org/wiki/xacro" >
     <xacro:include filename="inertial_macros.xacro"/>
-    <xacro:include filename="$(find robot_slam)/description/lidar.xacro"/>
-    <xacro:include filename="$(find robot_slam)/description/ros2_control.xacro"/>
     <material name="white">
         <color rgba="1 1 1 1" />
@@ -17,22 +15,20 @@
     </material>
     <link name="base_link">
+        <!-- Removed visual and collision boxes -->
+        <xacro:inertial_box mass="0.5" x="0.001" y="0.001" z="0.001">
+            <origin xyz="0 0 0" rpy="0 0 0"/>
+        </xacro:inertial_box>
     </link>
     <joint name="base_footprint_joint" type="fixed">
-        <parent link="base_link"/>
-        <child link="base_footprint"/>
-        <origin xyz="0 0 0" rpy="0 0 0"/>
+        <parent link="base_footprint"/>
+        <child link="base_link"/>
+        <origin xyz="0 0 0.037" rpy="0 0 0"/>
     </joint>
     <link name="base_footprint">
     </link>
-    <link name="odom"/>
-    <joint name="odom_to_base_link" type="fixed">
-        <parent link="odom"/>
-        <child link="base_link"/>
-        <origin xyz="0 0 0" rpy="0 0 0"/>
-    </joint>
     <joint name="container_joint" type="fixed">
         <parent link="base_link"/>
         <child link="container"/>
-        <origin xyz="-0.015 0 0.037"/>
+        <origin xyz="0 0 0" rpy="0 0 0"/>
     </joint>
     <link name="container">
@@ -54,30 +50,61 @@
         </xacro:inertial_box>
     </link>
-    <!-- Laser Link -->
-    <link name="laser">
+    <joint name="lidar_joint" type="fixed">
+        <parent link="base_link"/>
+        <child link="lidar"/>
+        <origin xyz="0 0 0.25" rpy="0 0 0"/>
+    </joint>
+    <link name="lidar">
         <visual>
             <geometry>
-                <cylinder radius="0.02" length="0.01"/>
+                <cylinder radius="0.035" length="0.058"/>
             </geometry>
-            <material name="black"/>
+            <material name="orange"/>
         </visual>
+        <collision>
+            <geometry>
+                <cylinder radius="0.035" length="0.058"/>
+            </geometry>
+        </collision>
+        <inertial>
+            <mass value="0.2"/>
+            <origin xyz="0 0 0.225" />
+            <inertia ixx="0.01" ixy="0.0" ixz="0.0" iyy="0.01" iyz="0.0" izz="0.01"/>
+        </inertial>
     </link>
-    <!-- Laser Joint -->
-    <joint name="laser_joint" type="fixed">
-        <parent link="base_link"/>
-        <child link="laser"/>
-        <origin xyz="0 0 0.1" rpy="0 0 0"/>
-    </joint>
     <!-- LEFT WHEEL LINK -->
     <joint name="left_wheel_joint" type="continuous">
         <parent link="base_link"/>
         <child link="left_wheel"/>
-        <origin xyz="0 0.085 0" rpy="-${pi/2} 0 0" />
-        <axis xyz="0 0 1"/>
+        <origin xyz="0 -0.1 0" rpy="${pi/2} 0 0" />
+        <axis xyz="0 0 -1"/>
     </joint>
     <link name="left_wheel">
         <visual>
             <geometry>
-                <cylinder radius="0.037" length="0.027"/>
+                <cylinder radius="0.035" length="0.027"/>
+            </geometry>
+            <material name="blue"/>
+        </visual>
+        <collision>
+            <geometry>
+                <cylinder radius="0.035" length="0.027"/>
+            </geometry>
+        </collision>
+        <xacro:inertial_cylinder mass="0.01" length="0.027" radius="0.035">
+            <origin xyz="0 0 0" rpy="0 0 0"/>
+        </xacro:inertial_cylinder>
+    </link>
+    <!-- RIGHT WHEEL LINK -->
+    <joint name="right_wheel_joint" type="continuous">
+        <parent link="base_link"/>
+        <child link="right_wheel"/>
+        <origin xyz="0 0.1 0" rpy="-${pi/2} 0 0" />
+        <axis xyz="0 0 1"/>
+    </joint>
+    <link name="right_wheel">
+        <visual>
+            <geometry>
+                <cylinder radius="0.035" length="0.027"/>
             </geometry>
             <material name="blue"/>
@@ -88,28 +115,5 @@
             </geometry>
         </collision>
-        <xacro:inertial_cylinder mass="0.01" length="0.027" radius="0.037">
-            <origin xyz="0 0 0" rpy="0 0 0"/>
-        </xacro:inertial_cylinder>
-    </link>
-    <!-- RIGHT WHEEL LINK -->
-    <joint name="right_wheel_joint" type="continuous">
-        <parent link="base_link"/>
-        <child link="right_wheel"/>
-        <origin xyz="0 -0.085 0" rpy="${pi/2} 0 0" />
-        <axis xyz="0 0 -1"/>
-    </joint>
-    <link name="right_wheel">
-        <visual>
-            <geometry>
-                <cylinder radius="0.037" length="0.027"/>
-            </geometry>
-            <material name="blue"/>
-        </visual>
-        <collision>
-            <geometry>
-                <cylinder radius="0.037" length="0.027"/>
-            </geometry>
-        </collision>
-        <xacro:inertial_cylinder mass="0.1" length="0.027" radius="0.037">
+        <xacro:inertial_cylinder mass="0.1" length="0.027" radius="0.035">
             <origin xyz="0 0 0" rpy="0 0 0"/>
         </xacro:inertial_cylinder>
@@ -158,32 +162,3 @@
         </xacro:inertial_sphere>
     </link>
-    <!-- ros2_control configuration -->
-    <ros2_control name="RealRobot" type="system">
-        <hardware>
-            <plugin>diffdrive_arduino/DiffDriveArduinoHardware</plugin>
-            <param name="left_wheel_name">left_wheel_joint</param>
-            <param name="right_wheel_name">right_wheel_joint</param>
-            <param name="loop_rate">30</param>
-            <param name="device">/dev/serial/by-path/platform-fd500000.pcie-pci-0000:01:00.0-usb-0:1.3:1.0-port0</param>
-            <param name="baud_rate">57600</param>
-            <param name="timeout_ms">1000</param>
-            <param name="enc_counts_per_rev">242</param>
-        </hardware>
-        <joint name="left_wheel_joint">
-            <command_interface name="velocity">
-                <param name="min">-50</param>
-                <param name="max">50</param>
-            </command_interface>
-            <state_interface name="position"/>
-            <state_interface name="velocity"/>
-        </joint>
-        <joint name="right_wheel_joint">
-            <command_interface name="velocity">
-                <param name="min">-50</param>
-                <param name="max">50</param>
-            </command_interface>
-            <state_interface name="position"/>
-            <state_interface name="velocity"/>
-        </joint>
-    </ros2_control>
 </robot>

File: robot_slam/description/ros2_control.xacro (robot description, xacro)
@@ -1,5 +1,5 @@
 <?xml version="1.0"?>
 <robot xmlns:xacro="http://www.ros.org/wiki/xacro">
-    <xacro>
+    <xacro:macro name="ros2_control_robot" params="use_ros2_control sim_mode">
         <ros2_control name="RealRobot" type="system">
             <hardware>
@@ -11,10 +11,10 @@
                 <param name="baud_rate">57600</param>
                 <param name="timeout_ms">1000</param>
-                <param name="enc_counts_per_rev">242</param>
+                <param name="enc_counts_per_rev">2194</param>
             </hardware>
             <joint name="left_wheel_joint">
                 <command_interface name="velocity">
-                    <param name="min">-50</param>
-                    <param name="max">50</param>
+                    <param name="min">-5</param>
+                    <param name="max">5</param>
                 </command_interface>
                 <state_interface name="position"/>
@@ -23,6 +23,6 @@
             <joint name="right_wheel_joint">
                 <command_interface name="velocity">
-                    <param name="min">-50</param>
-                    <param name="max">50</param>
+                    <param name="min">-5</param>
+                    <param name="max">5</param>
                 </command_interface>
                 <state_interface name="position"/>
@@ -30,4 +30,4 @@
             </joint>
         </ros2_control>
-    </xacro>
+    </xacro:macro>
 </robot>
